File: PCB/V3.0HackPad/V3.0HackPad.kicad_pcb (KiCad board)
At the start: 2 copper layers, 100 x 100 mm, 34 parts, among them SW1 RotaryEncoder, U1 Seeed Studio XIAO SAMD21

Commit message: Added some things and moved some things around
Updated some 3d models and moved a thew things around. :) But now I am finally done!!
Other:
- board text added: "Emre Kadir Tiren"
